File: pcb-arcade-controls/pcb-arcade-controls.kicad_sch (KiCad schematic)
At the start: 20 parts, among them J1 USB_C, SW1 SW_Push, U1 STM32F072CBT6, U3 XC6206, U4 USBLC6-2SC6

Commit message: PCB board wipe en connector toevoeging
Parts:
- added H1, H2, H3, H4: 10mm, arcade-controls:MountingHole_10mm, symbol Mechanical:MountingHole
- added IN1, IN10, IN11, IN12, IN13, IN14, IN15, IN16, IN17, IN18, IN19, IN2, IN20, IN21, IN22, IN23, IN24, IN3, IN4, IN5, IN6, IN7, IN8, IN9: Conn_01x02, Connector_PinHeader_2.54mm:PinHeader_1x02_P2.54mm_Vertical, symbol Connector_Generic:Conn_01x02
Connections:
- net A15: now also IN24.1 (Pin_1)
- net A4: now also IN1.1 (Pin_1)
- net A5: now also IN2.1 (Pin_1)
- net A6: now also IN3.1 (Pin_1)
- net A7: now also IN4.1 (Pin_1)
- net B0: now also IN5.1 (Pin_1)
- net B1: now also IN6.1 (Pin_1)
- net B10: now also IN8.1 (Pin_1)
- net B11: now also IN9.1 (Pin_1)
- net B12: now also IN10.1 (Pin_1)
- net B13: now also IN11.1 (Pin_1)
- net B14: now also IN12.1 (Pin_1)
- net B2: now also IN7.1 (Pin_1)
- net B3: now also IN23.1 (Pin_1)
- net B4: now also IN22.1 (Pin_1)
- net B5: now also IN21.1 (Pin_1)
- net B6: now also IN20.1 (Pin_1)
- net B7: now also IN19.1 (Pin_1)
- net B8: now also IN18.1 (Pin_1)
- net B9: now also IN17.1 (Pin_1)
- net C13: now also IN16.1 (Pin_1)
- net C14: now also IN15.1 (Pin_1)
- net C15: now also IN14.1 (Pin_1)
- net F0: now also IN13.1 (Pin_1)
- net GND: now also IN1.2 (Pin_2), IN10.2 (Pin_2), IN11.2 (Pin_2), IN12.2 (Pin_2), IN13.2 (Pin_2), IN14.2 (Pin_2), IN15.2 (Pin_2), IN16.2 (Pin_2), IN17.2 (Pin_2), IN18.2 (Pin_2), IN19.2 (Pin_2), IN2.2 (Pin_2), IN20.2 (Pin_2), IN21.2 (Pin_2), IN22.2 (Pin_2), IN23.2 (Pin_2), IN24.2 (Pin_2), IN3.2 (Pin_2), IN4.2 (Pin_2), IN5.2 (Pin_2), IN6.2 (Pin_2), IN7.2 (Pin_2), IN8.2 (Pin_2), IN9.2 (Pin_2)
Other:
- note added: "Inputs"
- note removed: "Matrix"
